File: Obstacle Course.sch (KiCad schematic (older format))
At the start: 15 parts

Commit message: Generated netlist
Parts:
- D1: renamed from D?; footprint (none) -> LEDs:LED_0805
- R1: renamed from R?; footprint (none) -> Resistors_SMD:R_0805
- R10, R11, R12, R13, R8, R9: renamed from R?; value R -> 0; footprint (none) -> Resistors_SMD:R_0603
- R2, R3, R4, R5, R6, R7: renamed from R?; footprint (none) -> Resistors_SMD:R_0603
- gave numbers to parts that had none: 1
Changed lines of the file:
@@
 $EndDescr
 $Comp
-L R R?
+L R R2
 U 1 1 586F3ED5
 P 2725 1750
-F 0 "R?" V 2805 1750 50  0000 C CNN
+F 0 "R2" V 2805 1750 50  0000 C CNN
 F 1 "0" V 2725 1750 50  0000 C CNN
-F 2 "" V 2655 1750 50  0000 C CNN
+F 2 "Resistors_SMD:R_0603" V 2655 1750 50  0001 C CNN
 F 3 "" H 2725 1750 50  0000 C CNN
 	1    2725 1750
@@
 $EndComp
 $Comp
-L R R?
+L R R3
 U 1 1 586F3FE7
 P 2725 2225
-F 0 "R?" V 2805 2225 50  0000 C CNN
+F 0 "R3" V 2805 2225 50  0000 C CNN
 F 1 "0" V 2725 2225 50  0000 C CNN
-F 2 "" V 2655 2225 50  0000 C CNN
+F 2 "Resistors_SMD:R_0603" V 2655 2225 50  0001 C CNN
 F 3 "" H 2725 2225 50  0000 C CNN
 	1    2725 2225
@@
 $EndComp
 $Comp
-L R R?
+L R R4
 U 1 1 586F400F
 P 2725 2725
-F 0 "R?" V 2805 2725 50  0000 C CNN
+F 0 "R4" V 2805 2725 50  0000 C CNN
 F 1 "0" V 2725 2725 50  0000 C CNN
-F 2 "" V 2655 2725 50  0000 C CNN
+F 2 "Resistors_SMD:R_0603" V 2655 2725 50  0001 C CNN
 F 3 "" H 2725 2725 50  0000 C CNN
 	1    2725 2725
@@
 $EndComp
 $Comp
-L R R?
+L R R5
 U 1 1 586F4040
 P 2725 3200
-F 0 "R?" V 2805 3200 50  0000 C CNN
+F 0 "R5" V 2805 3200 50  0000 C CNN
 F 1 "0" V 2725 3200 50  0000 C CNN
-F 2 "" V 2655 3200 50  0000 C CNN
+F 2 "Resistors_SMD:R_0603" V 2655 3200 50  0001 C CNN
 F 3 "" H 2725 3200 50  0000 C CNN
 	1    2725 3200
@@
 $EndComp
 $Comp
-L R R?
+L R R6
 U 1 1 586F4098
 P 2725 3675
-F 0 "R?" V 2805 3675 50  0000 C CNN
+F 0 "R6" V 2805 3675 50  0000 C CNN
 F 1 "0" V 2725 3675 50  0000 C CNN
-F 2 "" V 2655 3675 50  0000 C CNN
+F 2 "Resistors_SMD:R_0603" V 2655 3675 50  0001 C CNN
 F 3 "" H 2725 3675 50  0000 C CNN
 	1    2725 3675
@@
 $EndComp
 $Comp
-L R R?
+L R R7
 U 1 1 586F40D1
 P 2725 4150
-F 0 "R?" V 2805 4150 50  0000 C CNN
+F 0 "R7" V 2805 4150 50  0000 C CNN
 F 1 "0" V 2725 4150 50  0000 C CNN
-F 2 "" V 2655 4150 50  0000 C CNN
+F 2 "Resistors_SMD:R_0603" V 2655 4150 50  0001 C CNN
 F 3 "" H 2725 4150 50  0000 C CNN
 	1    2725 4150
@@
 $EndComp
 $Comp
-L R R?
+L R R8
 U 1 1 586F4117
 P 2725 4650
-F 0 "R?" V 2805 4650 50  0000 C CNN
-F 1 "R" V 2725 4650 50  0000 C CNN
-F 2 "" V 2655 4650 50  0000 C CNN
+F 0 "R8" V 2805 4650 50  0000 C CNN
+F 1 "0" V 2725 4650 50  0000 C CNN
+F 2 "Resistors_SMD:R_0603" V 2655 4650 50  0001 C CNN
 F 3 "" H 2725 4650 50  0000 C CNN
 	1    2725 4650
@@
 $EndComp
 $Comp
-L R R?
+L R R9
 U 1 1 586F4199
 P 2725 5175
-F 0 "R?" V 2805 5175 50  0000 C CNN
-F 1 "R" V 2725 5175 50  0000 C CNN
-F 2 "" V 2655 5175 50  0000 C CNN
+F 0 "R9" V 2805 5175 50  0000 C CNN
+F 1 "0" V 2725 5175 50  0000 C CNN
+F 2 "Resistors_SMD:R_0603" V 2655 5175 50  0001 C CNN
 F 3 "" H 2725 5175 50  0000 C CNN
 	1    2725 5175
@@
 $EndComp
 $Comp
-L R R?
+L R R10
 U 1 1 586F446D
 P 2725 5625
-F 0 "R?" V 2805 5625 50  0000 C CNN
-F 1 "R" V 2725 5625 50  0000 C CNN
-F 2 "" V 2655 5625 50  0000 C CNN
+F 0 "R10" V 2805 5625 50  0000 C CNN
+F 1 "0" V 2725 5625 50  0000 C CNN
+F 2 "Resistors_SMD:R_0603" V 2655 5625 50  0001 C CNN
 F 3 "" H 2725 5625 50  0000 C CNN
 	1    2725 5625
@@
 $EndComp
 $Comp
-L R R?
+L R R11
 U 1 1 586F44BA
 P 2725 6075
-F 0 "R?" V 2805 6075 50  0000 C CNN
-F 1 "R" V 2725 6075 50  0000 C CNN
-F 2 "" V 2655 6075 50  0000 C CNN
+F 0 "R11" V 2805 6075 50  0000 C CNN
+F 1 "0" V 2725 6075 50  0000 C CNN
+F 2 "Resistors_SMD:R_0603" V 2655 6075 50  0001 C CNN
 F 3 "" H 2725 6075 50  0000 C CNN
 	1    2725 6075
@@
 $EndComp
 $Comp
-L R R?
+L R R12
 U 1 1 586F44F8
 P 2725 6500
-F 0 "R?" V 2805 6500 50  0000 C CNN
-F 1 "R" V 2725 6500 50  0000 C CNN
-F 2 "" V 2655 6500 50  0000 C CNN
+F 0 "R12" V 2805 6500 50  0000 C CNN
+F 1 "0" V 2725 6500 50  0000 C CNN
+F 2 "Resistors_SMD:R_0603" V 2655 6500 50  0001 C CNN
 F 3 "" H 2725 6500 50  0000 C CNN
 	1    2725 6500
@@
 $EndComp
 $Comp
-L R R?
+L R R13
 U 1 1 586F4551
 P 2725 6925
-F 0 "R?" V 2805 6925 50  0000 C CNN
-F 1 "R" V 2725 6925 50  0000 C CNN
-F 2 "" V 2655 6925 50  0000 C CNN
+F 0 "R13" V 2805 6925 50  0000 C CNN
+F 1 "0" V 2725 6925 50  0000 C CNN
+F 2 "Resistors_SMD:R_0603" V 2655 6925 50  0001 C CNN
 F 3 "" H 2725 6925 50  0000 C CNN
 	1    2725 6925
@@
 $EndComp
 $Comp
-L Battery_Cell BT?
+L Battery_Cell BT1
 U 1 1 586F4A9F
 P 1275 2125
-F 0 "BT?" H 1375 2225 50  0000 L CNN
+F 0 "BT1" H 1375 2225 50  0000 L CNN
 F 1 "Battery_Cell" H 1375 2125 50  0000 L CNN
-F 2 "" V 1275 2185 50  0000 C CNN
+F 2 "" V 1275 2185 50  0001 C CNN
 F 3 "" V 1275 2185 50  0000 C CNN
 	1    1275 2125
@@
 	1275 7075 1275 2975
 $Comp
-L LED D?
+L LED D1
 U 1 1 586F58FE
 P 1275 2825
-F 0 "D?" H 1275 2925 50  0000 C CNN
+F 0 "D1" H 1275 2925 50  0000 C CNN
 F 1 "LED" H 1275 2725 50  0000 C CNN
-F 2 "" H 1275 2825 50  0000 C CNN
+F 2 "LEDs:LED_0805" H 1275 2825 50  0001 C CNN
 F 3 "" H 1275 2825 50  0000 C CNN
 	1    1275 2825
@@
 $EndComp
 $Comp
-L R R?
+L R R1
 U 1 1 586F5A77
 P 1275 2450
-F 0 "R?" V 1355 2450 50  0000 C CNN
+F 0 "R1" V 1355 2450 50  0000 C CNN
 F 1 "100" V 1275 2450 50  0000 C CNN
-F 2 "" V 1205 2450 50  0000 C CNN
+F 2 "Resistors_SMD:R_0805" V 1205 2450 50  0001 C CNN
 F 3 "" H 1275 2450 50  0000 C CNN
 	1    1275 2450
